File: prototype_WLCSP.sch (EAGLE design)
At the start: 8 parts

Commit message: update the file
Parts:
- removed S2: (no value), electron_v020:SPARK_TAC_SWITCHSMD
- added C1, C10, C2, C5: 2.2uF, electron_v020:SPARK_C-US
- added C11, C16, C8, C9: 10uF, electron_v020:BRETTS-SPARK-LIBRARY_C-US0603
- added C12, C13, C14: 0.1uF, electron_v020:SPARK_C-US
- added C3, C4: 12pF, electron_v020:SPARK_C-US
- added C6, C7: 20pF, electron_v020:SPARK_C-US
- added Q1: (no value), electron_v020:SPARK_Q_FC135
- added R1, R2, R3, R4: 10K, electron_v020:SPARK_R-US_
- added U$2: PARTICLE_TPS62291DRV, electron_v020:PARTICLE_TPS62291DRV
- added Y1: (no value), electron_v020:SPARKFUN-FREQCTRL_CRYSTAL5X3
- U$3: value SPARK_R-US_ -> 2.2uH; device electron_v020:SPARK_R-US_ -> electron_v020:PARTICLE_INDUCTORB
- U$4: value SPARK_R-US_ -> M18DPAD; device electron_v020:SPARK_R-US_ -> electron_v020:PARTICLE_M18DPAD
- U$5: value SPARK_C-US -> M18DPAD; device electron_v020:SPARK_C-US -> electron_v020:PARTICLE_M18DPAD
- U$6: value SPARK_C-US -> PARTICLE_DIODE_NT; device electron_v020:SPARK_C-US -> electron_v020:PARTICLE_DIODE_NT
Connections:
- removed net N$8: U$1.VSS_2, U$1.VSS_3, U$1.VSS_4, U$1.VSS_5
- new net !RST: U$5.17
- new net 5V: C8.1, JP1.VBUS, U$2.P$4, U$2.P$5, U$6.CATHODE
- new net A0: U$1.PC5, U$4.12
- new net A1: U$1.PC3, U$4.11
- new net A2: U$1.PC2, U$4.10
- new net A3: U$1.PA5, U$4.9
- new net A4: U$1.PA6, U$4.8
- new net A5: U$1.PA7, U$4.7
- new net B0: U$1.PC8, U$4.18
- new net B1: U$1.PC6, U$4.17
- new net B2: U$1.PB0, U$4.16
- new net B3: U$1.PB1, U$4.15
- new net B4: U$1.PC0, U$4.14
- new net B5: U$1.PC1, U$4.13
- new net C0: U$1.PD2, U$5.1
- new net C1: U$1.PC12, U$5.2
- new net C2: U$1.PC11, U$5.3
- new net C3: U$1.PC10, U$5.4
- new net C4: U$1.PB9, U$5.5
- new net C5: U$1.PB8, U$5.6
- new net D0: U$1.PB7, U$5.7
- new net D1: U$1.PB6, U$5.8
- new net D2: U$1.PB5, U$5.9
- new net D3: U$1.NJTRST/PB4, U$5.10
- new net D4: U$1.JTDO/TRACESSW0/PB3, U$5.11
- new net D5: U$1.JTDI/PA15, U$5.12
- new net D6: U$1.JTCK/SWCLK/PA14, U$5.13
- new net D7: U$1.JTMS/SWDIO/PA13, U$5.14
- new net DAC: U$1.PA4, U$4.6
- new net GND: C1.2, C10.2, C11.2, C12.2, C13.2, C14.2, C16.2, C2.2, C3.1, C4.1, C5.2, C6.2, C7.2, C8.2, C9.2, JP1.GND, S1.2, U$1.BOOT0, U$1.IRROFF, U$1.REGOFF, U$1.VSS_2, U$1.VSS_3, U$1.VSS_4, U$1.VSS_5, U$2.P$2, U$2.P$6, U$4.2, U$5.15
- new net N$11: C10.1, U$1.VREF+
- new net N$12: U$2.P$1, U$3.1
- new net N$3: C3.2, Q1.2, U$1.PC15
- new net N$4: C4.2, Q1.1, U$1.PC14
- new net N$7: C7.1, U$1.PH1/OSC_OUT, Y1.1
- new net N$9: C6.1, U$1.PH0/OSC_IN, Y1.2
- new net NRST: C5.1, R1.1, S1.4, U$1.NRST
- new net RX: U$1.PA10, U$4.4
- new net TX: U$1.PA9, U$4.3
- new net VBAT: R4.1, U$1.VBAT, U$5.16
- new net VIN: U$4.1, U$6.ANODE
- new net WKP: U$1.WKUP/PA0, U$4.5
- net +3V3: now also C11.1, C12.1, C13.1, C14.1, C16.1, C9.1, R1.2, R4.2, U$2.P$3, U$3.2, U$5.18; no longer U$1.VBAT
- net N$1: now also R2.1; no longer U$3.2
- net N$2: now also R3.1; no longer U$4.2
- net N$5: now also C2.1; no longer U$5.1
- net N$6: now also C1.1; no longer U$6.1
- net USB+: now also R2.2; no longer U$3.1
- net USB-: now also R3.2; no longer U$4.1
Other:
- moved on the sheet: S1
